Commit message: IMU 위치수정 0.108 -0.076 0.0

File: zetabank_robot_control/zetabank_description/urdf/zetabank.urdf.xacro (robot description, xacro)
@@ -75,5 +75,5 @@
     <parent link="base_link"/>
     <child link="imu_link"/>
-    <origin xyz="0.0 0.0 0.0" rpy="0 0 0"/>
+    <origin xyz="0.108 -0.076 0.0" rpy="0 0 0"/>
   </joint>
   <link name="imu_link"/>
